Commit message: refining files

File: janusseraphim_description/urdf/robots/janusseraphim.urdf (robot description, URDF)
Before this commit: robot my_robot, 10 links, 9 joints
Links:
- link base_link: geometry visual mesh filename=package://janusseraphim_description/meshes/grafika_100/visu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
- link ee_gear_link: geometry visual mesh filename=package://janusseraphim_description/meshes/grafika_100/visu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
- link ee_link: geometry visual mesh filename=package://janusseraphim_description/meshes/grafika_100/visu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
- link elbow_gear_link: geometry visual mesh filename=package://janusseraphim_description/meshes/grafika_100/visu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
- link elbow_link: geometry visual mesh filename=package://janusseraphim_description/meshes/grafika_100/visu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
- link elbow_servo_gear_link: geometry visual mesh filename=package://janusseraphim_description/meshes/grafika_100/visu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
- link rotator_link: geometry visual mesh filename=package://janusseraphim_description/meshes/grafika_100/visu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
- link shoulder_link: geometry visual mesh filename=package://janusseraphim_description/meshes/grafika_100/visu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
- link syringe_slider_link: geometry visual mesh filename=package://janusseraphim_description/meshes/grafika_100/visu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
- link wrist_link: geometry visual mesh filename=package://janusseraphim_description/meshes/grafika_100/visu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

Commit message: inverse kinematic is stil not perfect

File: janusseraphim_description/urdf/robots/janusseraphim.urdf (robot description, URDF)
Before this commit: robot my_robot, 10 links, 9 joints
Links:
- link base_link: geometry visual mesh filename=package://janusseraphim_description/meshes/janusseraphim_10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
- link ee_gear_link: geometry visual mesh filename=package://janusseraphim_description/meshes/janusseraphim_10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
- link ee_link: geometry visual mesh filename=package://janusseraphim_description/meshes/janusseraphim_10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
- link elbow_gear_link: geometry visual mesh filename=package://janusseraphim_description/meshes/janusseraphim_10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
- link elbow_link: geometry visual mesh filename=package://janusseraphim_description/meshes/janusseraphim_10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
- link elbow_servo_gear_link: geometry visual mesh filename=package://janusseraphim_description/meshes/janusseraphim_10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
- link rotator_link: geometry visual mesh filename=package://janusseraphim_description/meshes/janusseraphim_10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
- link shoulder_link: geometry visual mesh filename=package://janusseraphim_description/meshes/janusseraphim_10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
- link syringe_slider_link: geometry visual mesh filename=package://janusseraphim_description/meshes/janusseraphim_10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
- link wrist_link: geometry visual mesh filename=package://janusseraphim_description/meshes/janusseraphim_10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
